Commit message: cac_description: rebuild from NEW JOINTS KESHAV ASSEMBLY.step (new joints)
Only the robot's right side has the new joints in this CAD, so the left
is rebuilt as its exact mirror (rods, joints, wheels, pivots; body and
diff bar untouched). prep_keshav.py rotates the file's frame into the
generator's convention, drops a duplicated motor cap and bogie block and
sub-1 cm^3 hardware, and assigns links and materials. Masses from the
team's materials (PLA joints, carbon-fibre rods as 20x16 mm tubes) plus
assumed motors/wheels/body: 21.0 kg. Standing: 1.11 x 0.75 x 0.68 m,
body level (0.5 deg; the old CAD gave 6), all six wheels on the ground.
Width 0.7505 m with the mirrored side: 0.5 mm over 0.75 m.

File: src/cac_description/urdf/rover.urdf (robot description, URDF)
Before this commit: robot vanguard_rover, 13 links, 12 joints
Links:
- link base_link: mass 4.45526 -> 4.62879; geometry collision box size=0.0599379 0.060058 0.0713146; collision box size=0.0606425 0.0640065 0.0625382
- link diff_bar: mass 1.17923 -> 0.722942; geometry collision box size=0.0566059 0.0802922 0.644069; visual mesh filename=package://cac_description/meshes/diff_bar.stl
- link left_bogie: mass 5.07065 -> 2.93299; geometry collision box size=0.00500342 0.0574711 0.101621; collision box size=0.00500444 0.0574711 0.101621
- link left_rocker: mass 3.03678 -> 1.85956; geometry collision box size=0.0199525 0.019978 0.284203; collision box size=0.0200247 0.0206169 0.24702
- link right_bogie: mass 5.07026 -> 2.93299; geometry collision box size=0.00500342 0.0574711 0.101621; collision box size=0.00500444 0.0574711 0.101621
- link right_rocker: mass 3.01782 -> 1.85956; geometry collision box size=0.0199525 0.019978 0.284203; collision box size=0.0200247 0.0206169 0.24702
Joints:
- joint base_footprint_joint: origin xyz=0 0 0.719964 rpy=0 0.104545 0 -> xyz=0 0 0.486533 rpy=0 -0.0088856 0
- joint diff_bar_joint: mimic joint=right_rocker_joint multiplier=0.412439 offset=0 -> joint=right_rocker_joint multiplier=0.411765 offset=0; origin xyz=-0.0941 -5.55112e-17 0.143 rpy=0 0 0 -> xyz=-0.094 0.000309387 0.1 rpy=0 0 0
- joint left_bogie_joint: origin xyz=0.5159 0.0225 -0.1793 rpy=0 0 0 -> xyz=0.35 0 -0.122 rpy=0 0 0
- joint left_front_wheel_joint: origin xyz=0.415178 -0.01725 -0.3361 rpy=0 0 0 -> xyz=0.187462 -0.0201906 -0.259324 rpy=0 0 0
- joint left_middle_wheel_joint: origin xyz=-0.336107 -0.01725 -0.415159 rpy=0 0 0 -> xyz=-0.334174 -0.0201906 -0.254698 rpy=0 0 0
- joint left_rear_wheel_joint: origin xyz=-0.221009 0.00525 -0.636502 rpy=0 0 0 -> xyz=-0.348647 -0.0201906 -0.37345 rpy=0 0 0
- joint left_rocker_joint: origin xyz=0 0.28 0 rpy=0 0 0 -> xyz=0 0.343691 0 rpy=0 0 0
- joint right_bogie_joint: origin xyz=0.5225 -0.0225 -0.1731 rpy=0 0 0 -> xyz=0.35 0 -0.122 rpy=0 0 0
- joint right_front_wheel_joint: origin xyz=0.408712 0.01775 -0.34272 rpy=0 0 0 -> xyz=0.187462 0.0201906 -0.259324 rpy=0 0 0
- joint right_middle_wheel_joint: origin xyz=-0.342601 0.01775 -0.421498 rpy=0 0 0 -> xyz=-0.334174 0.0201906 -0.254698 rpy=0 0 0
- joint right_rear_wheel_joint: origin xyz=-0.221009 -0.00475001 -0.636502 rpy=0 0 0 -> xyz=-0.348647 0.0201906 -0.37345 rpy=0 0 0
- joint right_rocker_joint: origin xyz=0 -0.28 0 rpy=0 0 0 -> xyz=0 -0.343691 0 rpy=0 0 0

File: src/cac_description/urdf/rover_sim.urdf (robot description, URDF)
Before this commit: robot vanguard_rover, 13 links, 12 joints
Links:
- link base_link: mass 4.45526 -> 4.62879; geometry collision box size=0.0599379 0.060058 0.0713146; collision box size=0.0606425 0.0640065 0.0625382
- link diff_bar: mass 1.17923 -> 0.722942; geometry collision box size=0.0566059 0.0802922 0.644069; visual mesh filename=package://cac_description/meshes/diff_bar.stl
- link left_bogie: mass 5.07065 -> 2.93299; geometry collision box size=0.00500342 0.0574711 0.101621; collision box size=0.00500444 0.0574711 0.101621
- link left_rocker: mass 3.03678 -> 1.85956; geometry collision box size=0.0199525 0.019978 0.284203; collision box size=0.0200247 0.0206169 0.24702
- link right_bogie: mass 5.07026 -> 2.93299; geometry collision box size=0.00500342 0.0574711 0.101621; collision box size=0.00500444 0.0574711 0.101621
- link right_rocker: mass 3.01782 -> 1.85956; geometry collision box size=0.0199525 0.019978 0.284203; collision box size=0.0200247 0.0206169 0.24702
Joints:
- joint base_footprint_joint: origin xyz=0 0 0.719964 rpy=0 0.104545 0 -> xyz=0 0 0.486533 rpy=0 -0.0088856 0
- joint diff_bar_joint: origin xyz=-0.0941 -5.55112e-17 0.143 rpy=0 0 0 -> xyz=-0.094 0.000309387 0.1 rpy=0 0 0
- joint left_bogie_joint: origin xyz=0.5159 0.0225 -0.1793 rpy=0 0 0 -> xyz=0.35 0 -0.122 rpy=0 0 0
- joint left_front_wheel_joint: origin xyz=0.415178 -0.01725 -0.3361 rpy=0 0 0 -> xyz=0.187462 -0.0201906 -0.259324 rpy=0 0 0
- joint left_middle_wheel_joint: origin xyz=-0.336107 -0.01725 -0.415159 rpy=0 0 0 -> xyz=-0.334174 -0.0201906 -0.254698 rpy=0 0 0
- joint left_rear_wheel_joint: origin xyz=-0.221009 0.00525 -0.636502 rpy=0 0 0 -> xyz=-0.348647 -0.0201906 -0.37345 rpy=0 0 0
- joint left_rocker_joint: origin xyz=0 0.28 0 rpy=0 0 0 -> xyz=0 0.343691 0 rpy=0 0 0
- joint right_bogie_joint: origin xyz=0.5225 -0.0225 -0.1731 rpy=0 0 0 -> xyz=0.35 0 -0.122 rpy=0 0 0
- joint right_front_wheel_joint: origin xyz=0.408712 0.01775 -0.34272 rpy=0 0 0 -> xyz=0.187462 0.0201906 -0.259324 rpy=0 0 0
- joint right_middle_wheel_joint: origin xyz=-0.342601 0.01775 -0.421498 rpy=0 0 0 -> xyz=-0.334174 0.0201906 -0.254698 rpy=0 0 0
- joint right_rear_wheel_joint: origin xyz=-0.221009 -0.00475001 -0.636502 rpy=0 0 0 -> xyz=-0.348647 0.0201906 -0.37345 rpy=0 0 0
- joint right_rocker_joint: origin xyz=0 -0.28 0 rpy=0 0 0 -> xyz=0 -0.343691 0 rpy=0 0 0

Commit message: cac_description: per-material visuals (white PLA, black CF, wood diff bar)
Each link is now drawn per material in colours that follow the team's
renders: PLA joints white, carbon-fibre rods black, rubber wheels, alu
body, wooden differential bar, steel pins, dark motors. Combined per-link
meshes stay for tools/tests. Material colour names are prefixed (mat_)
because a duplicate material name made urdfdom reject the file; a test
now checks names are unique. README: how to drop the rover into the
cac_sim arena.

File: src/cac_description/urdf/rover.urdf (robot description, URDF)
Before this commit: robot vanguard_rover, 13 links, 12 joints
Links:
- link base_link: geometry collision box size=0.0599379 0.060058 0.0713146; collision box size=0.0606425 0.0640065 0.0625382
- link diff_bar: mass 0.722942 -> 0.584601; geometry collision box size=0.0566059 0.0802922 0.644069; visual mesh filename=package://cac_description/meshes/diff_bar__pla.stl
- link left_bogie: geometry collision box size=0.00500342 0.0574711 0.101621; collision box size=0.00500444 0.0574711 0.101621
- link left_rocker: geometry collision box size=0.0199525 0.019978 0.284203; collision box size=0.0200247 0.0206169 0.24702
- link right_bogie: geometry collision box size=0.00500342 0.0574711 0.101621; collision box size=0.00500444 0.0574711 0.101621
- link right_rocker: geometry collision box size=0.0199525 0.019978 0.284203; collision box size=0.0200247 0.0206169 0.24702

File: src/cac_description/urdf/rover_sim.urdf (robot description, URDF)
Before this commit: robot vanguard_rover, 13 links, 12 joints
Links:
- link base_link: geometry collision box size=0.0599379 0.060058 0.0713146; collision box size=0.0606425 0.0640065 0.0625382
- link diff_bar: mass 0.722942 -> 0.584601; geometry collision box size=0.0566059 0.0802922 0.644069; visual mesh filename=package://cac_description/meshes/diff_bar__pla.stl
- link left_bogie: geometry collision box size=0.00500342 0.0574711 0.101621; collision box size=0.00500444 0.0574711 0.101621
- link left_rocker: geometry collision box size=0.0199525 0.019978 0.284203; collision box size=0.0200247 0.0206169 0.24702
- link right_bogie: geometry collision box size=0.00500342 0.0574711 0.101621; collision box size=0.00500444 0.0574711 0.101621
- link right_rocker: geometry collision box size=0.0199525 0.019978 0.284203; collision box size=0.0200247 0.0206169 0.24702

Commit message: cac_description: tight collision boxes; rocker clamp parts; review fixes
Independent review found the PCA collision boxes tilted on hollow parts:
collision envelope 0.856 m wide vs 0.7505 m real, body box 95 mm below
the body. Now each part uses the axis-aligned box unless the PCA box is
smaller and stays within its bounds, and hollow parts over 1 L are split
into up to 8 boxes: envelope 0.7325 m wide, lowest point at the visual's.
Component130/141/142 clamp the rocker rod and move to the rocker.
Tests: mimic multipliers and signs, L/R symmetry, boxes within visual
bounds, envelope width and lowest point, README mass vs build summary.
Docs and generated header no longer name the old CAD.

File: src/cac_description/urdf/rover.urdf (robot description, URDF)
Before this commit: robot vanguard_rover, 13 links, 12 joints
Links:
- link base_link: geometry collision box size=0.00612834 0.03 0.00800002; collision box size=0.00612834 0.03 0.00800002
- link diff_bar: geometry collision box size=0.05 0.644068 0.0761355; visual mesh filename=package://cac_description/meshes/diff_bar__pla.stl
- link left_bogie: mass 2.93299 -> 2.88492; geometry collision box size=0.0200138 0.0201369 0.183185; collision box size=0.020871 0.0200713 0.117692
- link left_rocker: mass 1.85956 -> 1.90763; geometry collision box size=0.0199525 0.019978 0.284203; collision box size=0.0200247 0.0206169 0.24702
- link right_bogie: mass 2.93299 -> 2.88492; geometry collision box size=0.0200138 0.0201369 0.183185; collision box size=0.020871 0.0200713 0.117692
- link right_rocker: mass 1.85956 -> 1.90763; geometry collision box size=0.0199525 0.019978 0.284203; collision box size=0.0200247 0.0206169 0.24702

File: src/cac_description/urdf/rover_sim.urdf (robot description, URDF)
Before this commit: robot vanguard_rover, 13 links, 12 joints
Links:
- link base_link: geometry collision box size=0.00612834 0.03 0.00800002; collision box size=0.00612834 0.03 0.00800002
- link diff_bar: geometry collision box size=0.05 0.644068 0.0761355; visual mesh filename=package://cac_description/meshes/diff_bar__pla.stl
- link left_bogie: mass 2.93299 -> 2.88492; geometry collision box size=0.0200138 0.0201369 0.183185; collision box size=0.020871 0.0200713 0.117692
- link left_rocker: mass 1.85956 -> 1.90763; geometry collision box size=0.0199525 0.019978 0.284203; collision box size=0.0200247 0.0206169 0.24702
- link right_bogie: mass 2.93299 -> 2.88492; geometry collision box size=0.0200138 0.0201369 0.183185; collision box size=0.020871 0.0200713 0.117692
- link right_rocker: mass 1.85956 -> 1.90763; geometry collision box size=0.0199525 0.019978 0.284203; collision box size=0.0200247 0.0206169 0.24702

Commit message: cac_description: RealSense D455 on a printed bracket, at the studied pose
Pose from a ray-cast study over positions and pitches against the
rover's real geometry: x 0.35, z 0.68 m, 22.5 deg down; 0% self-
occlusion, blind zone 0.24 m past the front wheels, 99% of the 0.6-4 m
band, 40 x 6 cm crater visible from ~2.4 m, ArUco boards in view to 8 m
(11 deg margin). Bracket: one PLA part (FreeCAD source tools/
d455_bracket.py, STEP+STL in cad/): saddle on the front top 30x30
member with 2 x M5, web, 23 deg plate with 1/4-20 hole and anti-rotation
lip. URDF: camera_mount + camera_link + optical frames; Gazebo colour
camera + depth camera (the gz-sim 8 rgbd_camera renders colour unlit).
Simulated frames verified in the arena.

File: src/cac_description/urdf/rover.urdf (robot description, URDF)
Before this commit: robot vanguard_rover, 13 links, 12 joints
Links:
- added link camera_color_optical_frame
- added link camera_depth_optical_frame
- added link camera_link, mass 0.39; collision box size=0.026 0.124 0.029; visual box size=0.026 0.124 0.029
- added link camera_mount, mass 0.0964527; collision box size=0.118642 0.07 0.130437; visual mesh filename=package://cac_description/meshes/camera_mount.stl
Joints:
- added joint camera_color_optical_joint: type fixed, parent camera_link, child camera_color_optical_frame, origin xyz=0 0 0 rpy=-1.5708 0 -1.5708
- added joint camera_depth_optical_joint: type fixed, parent camera_link, child camera_depth_optical_frame, origin xyz=0 0 0 rpy=-1.5708 0 -1.5708
- added joint camera_joint: type fixed, parent camera_mount, child camera_link, origin xyz=0.3517 0 0.1903 rpy=0 0.40158 0
- added joint camera_mount_joint: type fixed, parent base_link, child camera_mount, origin xyz=0 0 0 rpy=0 0 0

File: src/cac_description/urdf/rover_sim.urdf (robot description, URDF)
Before this commit: robot vanguard_rover, 13 links, 12 joints
Links:
- added link camera_color_optical_frame
- added link camera_depth_optical_frame
- added link camera_link, mass 0.39; collision box size=0.026 0.124 0.029; visual box size=0.026 0.124 0.029
- added link camera_mount, mass 0.0964527; collision box size=0.118642 0.07 0.130437; visual mesh filename=package://cac_description/meshes/camera_mount.stl
Joints:
- added joint camera_color_optical_joint: type fixed, parent camera_link, child camera_color_optical_frame, origin xyz=0 0 0 rpy=-1.5708 0 -1.5708
- added joint camera_depth_optical_joint: type fixed, parent camera_link, child camera_depth_optical_frame, origin xyz=0 0 0 rpy=-1.5708 0 -1.5708
- added joint camera_joint: type fixed, parent camera_mount, child camera_link, origin xyz=0.3517 0 0.1903 rpy=0 0.40158 0
- added joint camera_mount_joint: type fixed, parent base_link, child camera_mount, origin xyz=0 0 0 rpy=0 0 0

Commit message: cac_description: D455 bracket fixes from the mechanical review
Saddle had 0.00 mm clearance on the 30x30 member: 0.3 mm per side
fore-aft now. M5 bolts moved up to bear on the member (anti-rotation, 6 mm
ligament). Tripod hole 2.8 mm behind the camera centre (realsense-ros
d455 mount offset) so the body centre lands on the URDF pose; the lip
clears it (FreeCAD overlap 0). Plate and web 40 mm wide: prints without
supports. README: PETG/ASA (PLA creeps), M5x50 + fender washers + nyloc
<= 1 N m, 1/4-20 x 3/8 in screw. Depth optical frame and sensor moved to
the left imager (+47.5 mm y).

File: src/cac_description/urdf/rover.urdf (robot description, URDF)
Before this commit: robot vanguard_rover, 17 links, 16 joints
Links:
- link camera_mount: mass 0.0964527 -> 0.119932; geometry collision box size=0.121243 0.06 0.131414; visual mesh filename=package://cac_description/meshes/camera_mount.stl
Joints:
- joint camera_depth_optical_joint: origin xyz=0 0 0 rpy=-1.5708 0 -1.5708 -> xyz=0 0.0475 0 rpy=-1.5708 0 -1.5708

File: src/cac_description/urdf/rover_sim.urdf (robot description, URDF)
Before this commit: robot vanguard_rover, 17 links, 16 joints
Links:
- link camera_mount: mass 0.0964527 -> 0.119932; geometry collision box size=0.121243 0.06 0.131414; visual mesh filename=package://cac_description/meshes/camera_mount.stl
Joints:
- joint camera_depth_optical_joint: origin xyz=0 0 0 rpy=-1.5708 0 -1.5708 -> xyz=0 0.0475 0 rpy=-1.5708 0 -1.5708
